File: Pcb/ControleurPulve_kicad/ControleurPulve.kicad_sch (KiCad schematic)
At the start: 16 parts, among them J1 Debitmètre Gauche, J2 Débitmètre Droit, J3 GPS, J4 Conn_G, J5 Capteur de pression, J6 12V, J7 Conn_D, U2 LM2596S-5, U3 PC817, U4 PC817

Commit message: Avancement schematic
Parts:
- removed C1: 680µF, Capacitor_SMD:CP_Elec_10x10.5, symbol Device:C_Polarized
- removed C2: 220µF, Capacitor_SMD:CP_Elec_6.3x5.4, symbol Device:C_Polarized
- removed D1: 1N5821, Diode_THT:D_DO-201AD_P12.70mm_Horizontal, symbol Diode:1N5821
- removed J1: Debitmètre Gauche, mesEmpreintes:TerminalBlock_bornier-3_P5.08mm, symbol Connector:Screw_Terminal_01x03
- removed J2: Débitmètre Droit, mesEmpreintes:TerminalBlock_bornier-3_P5.08mm, symbol Connector:Screw_Terminal_01x03
- removed J3: GPS, Connector_PinSocket_2.54mm:PinSocket_1x05_P2.54mm_Vertical, symbol Connector_Generic:Conn_01x05
- removed J4: Conn_G, Connector_PinSocket_2.54mm:PinSocket_1x15_P2.54mm_Vertical, symbol Connector_Generic:Conn_01x15
- removed J5: Capteur de pression, Connector_PinHeader_2.54mm:PinHeader_1x03_P2.54mm_Vertical, symbol Connector_Generic:Conn_01x03
- removed J6: 12V, mesEmpreintes:TerminalBlock_bornier-2_P5.08mm, symbol Connector:Screw_Terminal_01x02
- removed J7: Conn_D, Connector_PinSocket_2.54mm:PinSocket_1x15_P2.54mm_Vertical, symbol Connector_Generic:Conn_01x15
- removed L1: 33µH, Inductor_SMD:L_Changjiang_FXL0650, symbol Device:L
- removed R1, R2: 10k, Resistor_SMD:R_0603_1608Metric, symbol Device:R
- removed U2: LM2596S-5, Package_TO_SOT_SMD:TO-263-5_TabPin3, symbol Regulator_Switching:LM2596S-5
- removed U3, U4: PC817, mesEmpreintes:OPTO-SMD4, symbol Isolator:PC817
- added C10, C11, C4, C5, C6, C7, C8: C, Capacitor_SMD:C_0805_2012Metric, symbol Device:C
- added C12, C13, C14, C15: 10nF, Capacitor_SMD:C_0603_1608Metric, symbol Device:C
- added C3, C9: C_Polarized, Capacitor_SMD:CP_Elec_8x10, symbol Device:C_Polarized
- added D2: MRA4004T3G, Diode_SMD:D_SMA, symbol Diode:MRA4004T3G
- added D7: LESD5D5.0CT1G, Diode_SMD:D_SOD-523, symbol Diode:ESD5Zxx
- added F1: MINISMDC050F-2, Diode_SMD:D_1812_4532Metric_Pad1.30x3.40mm_HandSolder, symbol Device:Polyfuse
- added J10: Débitmètre Droit, mesEmpreintes:TerminalBlock_bornier-3_P5.08mm, symbol Connector:Screw_Terminal_01x03
- added J11: Screw_Terminal_01x02, TerminalBlock_RND:TerminalBlock_RND_205-00287_1x02_P5.08mm_Horizontal, symbol Connector:Screw_Terminal_01x02
- added J12: GPS, Connector_PinSocket_2.54mm:PinSocket_1x05_P2.54mm_Vertical, symbol Connector_Generic:Conn_01x05
- added J13: Analogique 0-3.3V, Connector_PinHeader_2.54mm:PinHeader_1x03_P2.54mm_Vertical, symbol Connector_Generic:Conn_01x03
- added J14: Screw_Terminal_01x02, symbol Connector:Screw_Terminal_01x02
- added J8: Barrel_Jack_MountingPin, Connector_BarrelJack:BarrelJack_Horizontal, symbol Connector:Barrel_Jack_MountingPin
- added J9: Debitmètre Gauche, mesEmpreintes:TerminalBlock_bornier-3_P5.08mm, symbol Connector:Screw_Terminal_01x03
- added JP1, JP2: SolderJumper_3_Open, Jumper:SolderJumper-3_P1.3mm_Open_Pad1.0x1.5mm, symbol Jumper:SolderJumper_3_Open
- added R3, R4: 10k, Resistor_SMD:R_0603_1608Metric, symbol Device:R
- added R5: 150R .1%, Resistor_SMD:R_1206_3216Metric, symbol Device:R
- added R9: 10k, Resistor_SMD:R_0603_1608Metric_Pad0.98x0.95mm_HandSolder, symbol Device:R
- added U5, U6: PC817, mesEmpreintes:OPTO-SMD4, symbol Isolator:PC817
- added U7: R-78E3.3-0.5/K7805-1000R3, Converter_DCDC:Converter_DCDC_RECOM_RPMx.x-x.0, symbol Regulator_Switching:R-78E3.3-0.5
- added U8: ESP32_C3_supermini, ESP_modules:module, symbol ESP32-Modules:ESP32_C3_supermini
- added U9: TPS22810DBVR, TPS22810:DBV0006A_L, symbol TPS22810:TPS22810DBVR
Connections:
- net GND: now also C10.2, C11.2, C12.2, C13.2, C14.2, C15.2, C3.2, C4.2, C7.2, C8.2, C9.2, J10.2 (Pin_2), J11.2 (Pin_2), J12.2 (Pin_2), J13.3 (Pin_3), J8.2, J8.MP (MountPin), J9.2 (Pin_2), R5.2, U5.3, U6.3, U7.2 (GND), U8.13 (GND), U9.2 (GND)
- new net: J10.1 (Pin_1), U6.2
- new net: C7.1, D2.2 (A), J11.1 (Pin_1), J8.1
- new net: J14.2 (Pin_2), JP1.1 (A), R5.1
- new net: J9.1 (Pin_1), U5.2
- new net: C14.1, U9.4 (CT)
- new net: C11.1, J12.1 (Pin_1), JP2.2 (C)
- new net: R9.2, U9.3 (EN_UVLO)
- new net: C15.1, J13.1 (Pin_1), JP1.3 (B)
- new net: D2.1 (K), F1.1
- new net 12V: C10.1, C3.1, C4.1, C9.1, F1.2, R9.1, U7.1 (IN), U9.1 (VIN)
- new net 12V_OUT: J10.3 (Pin_3), J14.1 (Pin_1), J9.3 (Pin_3), U5.1, U6.1, U9.6 (VOUT)
- new net 3V3: R3.2, R4.2
- new net 3V3_OUT: JP2.1 (A), U8.12 (VCC_3V3)
- new net 5V: C12.1, C13.1, C5.1, C6.1, C8.1, D7.1 (K), J13.2 (Pin_2), JP2.3 (B), U7.3 (OUT), U8.14 (VUSB)
- new net debit_droit: R4.1, U6.4
- new net debit_gauche: R3.1, U5.4
- new net pression: JP1.2 (C)
- no-connect marks 23 -> 1
Other:
- note added: "0-3.3V"
- note added: "4-20"
- note added: "Avec 150 Ω : 4 mA → 0,004 A × 150 Ω = 0,6 V 20 mA → 0,02 A × 150 Ω = 3,0 V"
- note added: "DebitDouille V2.0 06/25"
- note added: "Debitmetres"
- note added: "GPS neo7M"
- note added: "General : pins debug, percages, etc"
- note added: "Microcontroleur"
- note added: "Nicolas DAUY - FURGO"
- note added: "POWER"
- note added: "Power Pins 5V - This is 5v out from the USB port. You can also use this as a voltage input but you must have some sort of diode (schottky, signal, power) between your external power source and this pin with anode to battery, cathode to 5V pin. 3V3 - This is the regulated output from the onboard regulator. You can draw 700mA GND - Power/data/signal ground Strapping Pins According to the chip manua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"
- note added: "Pression --> analog ou 4-20 au choix"
